File: turing-machine.kicad_pcb (KiCad board)
At the start: 2 copper layers, 50.5 x 241 mm, 123 parts, among them J1 Conn_02x05_Odd_Even, J2 cv, J3 clock, J4 out, J5 noise, J6 Conn_02x08_Odd_Even, J7 Conn_02x08_Odd_Even, J8 pulse, Q1 BC547, SW1 SW_Rotary12, SW2 SW_SPDT_MSM, U1 TL072, U10 4050, U11 L78L09_SOT89, U12 4081, U13 4081, U14 TL072, U2 DAC08, U3 TL431DBZ, U4 4016, U5 TL072, U6 4015, U7 4015, U8 L78L09_SOT89, U9 4050

Commit message: ready for v1 manu
Parts:
- removed C16, C17, C18: 1n, Capacitor_SMD:C_0805_2012Metric
- removed the C3 at (59.5, 67.4)
- removed the C5 at (82.5, 70.3)
- added D14: 1N4148, Diode_SMD:D_SOD-323_HandSoldering, F.Cu at (78.1, 60.7)
- added H24: trim, Eurorack:Mech-LED-Hole-3mm, F.Cu at (64.9, 195.4)
- added Q2: BCM847, Package_SO:TSOP-6_1.65x3.05mm_P0.95mm, F.Cu at (81.7, 66.2)
- added R34: 10K, Resistor_SMD:R_0805_2012Metric, F.Cu at (69.3, 54.8)
- R10: value 15K -> 10K
- R11: value 68K -> 100K
- R12: value 10K -> 3.9K
- R30: value 10K -> 68K
- R31: value 10K -> 15K
- R32: value 10K -> 470K
- R7: value 15K -> 100K
- R8: value 100K -> 8.2K
- R9: value 470K -> 470
- RV3: moved to F.Cu
- U2: value DAC08 -> DAC0800_SOIC
- moved R30 37.7 mm to (87.3, 74.5), turned to 0 degrees
- moved D3 26.6 mm to (58.7, 65.8), turned to 90 degrees
- moved R31 26.2 mm to (87.3, 72.1), turned to 180 degrees
- moved R8 24.4 mm to (83.0, 63.0)
- moved R14 10.1 mm to (68.3, 14.0), turned to -90 degrees
- moved R11 8.13 mm to (82.5, 70.3), turned to -90 degrees
- moved R15 7.39 mm to (70.9, 14.0), turned to 90 degrees
- moved R10 6.10 mm to (85.1, 66.6), turned to -90 degrees
- moved R16 5.86 mm to (73.4, 14.0), turned to 90 degrees
- moved U3 5.67 mm to (72.1, 18.3), turned to 0 degrees
- moved R12 5.11 mm to (78.4, 66.1), turned to -90 degrees
- moved R32 4.95 mm to (75.8, 66.1), turned to -90 degrees
- moved C5 4.04 mm to (75.9, 14.0), turned to 90 degrees
- moved C3 3.44 mm to (84.6, 77.7)
- moved C4 3.26 mm to (78.5, 14.0), turned to -90 degrees
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- renumbered C12 to C10, C13 to C11, C14 to C12, C15 to C13, C4 to C3, C6 to C4, C7 to C5, C8 to C6, C9 to C7, C10 to C8, C11 to C9
Connections:
- C5 pad 1: Net-(U2-CMP) -> -12V
- C5 pad 2: -12V -> Net-(U2-COMPEN)
- D3 pad 1: /CLK' -> Net-(D3-K)
- D3 pad 2: Net-(D3-A) -> GND
- R10 pad 1: Net-(U1A--) -> Net-(Q2A-C1)
- R10 pad 2: GND -> Net-(Q2B-B2)
- R11 pad 1: +12V -> Net-(Q2B-B2)
- R11 pad 2: Net-(U1A--) -> GND
- R12 pad 1: /CLK' -> +12V
- R12 pad 2: GND -> Net-(Q2B-C2)
- R15 pad 1: Net-(U2-R+) -> Net-(U3-K)
- R15 pad 2: Net-(U3-K) -> Net-(U2-VREF+)
- R16 pad 2: Net-(U2-R-) -> Net-(U2-VREF-)
- R30 pad 1: /B4' -> Net-(U1A--)
- R30 pad 2: Net-(U6B-D) -> +12V
- R31 pad 1: /B0' -> GND
- R31 pad 2: Net-(U7A-D) -> Net-(U1A--)
- R32 pad 1: /s12' -> /CLK'
- R32 pad 2: Net-(U7B-D) -> Net-(Q2B-C2)
- R7 pad 1: Net-(U1A-+) -> Net-(D3-K)
- R8 pad 1: Net-(U1A-+) -> +12V
- R8 pad 2: GND -> Net-(Q2A-C1)
- R9 pad 1: Net-(U1A-+) -> GND
- R9 pad 2: /CLK' -> Net-(Q2A-E1)
- U1 pad 1: Net-(D3-A) -> Net-(D14-A)
- U1 pad 3: Net-(U1A-+) -> Net-(Q2B-C2)
- U2 pad 1: GND -> +12V
- U2 pad 10: /B5' -> /B1'
- U2 pad 11: /B6' -> /B2'
- U2 pad 12: /B7' -> /B3'
- U2 pad 13: +12V -> /B4'
- U2 pad 14: Net-(U2-R+) -> /B5'
- U2 pad 15: Net-(U2-R-) -> /B6'
- U2 pad 16: Net-(U2-CMP) -> /B7'
- U2 pad 2: GND -> Net-(U2-VREF+)
- U2 pad 3: -12V -> Net-(U2-VREF-)
- U2 pad 4: Net-(U1B--) -> Net-(U2-COMPEN)
- U2 pad 5: /B0' -> GND
- U2 pad 6: /B1' -> GND
- U2 pad 7: /B2' -> -12V
- U2 pad 8: /B3' -> Net-(U1B--)
- U2 pad 9: /B4' -> /B0'
- U6 pad 15: Net-(U6B-D) -> /B4'
- U7 pad 15: Net-(U7B-D) -> /s12'
- U7 pad 7: Net-(U7A-D) -> /B0'
Routing:
- net GND: track 287.9 -> 341.7 mm, vias 27 -> 29
- net Net-(U1A-+): track 32.2 -> 0.00 mm
- net Net-(D3-K): track 0.00 -> 25.7 mm
- net Net-(D14-A): track 0.00 -> 19.9 mm
- net +12V: track 336.9 -> 352.2 mm
- net Net-(Q2B-C2): track 0.00 -> 11.9 mm
- net -12V: track 213.8 -> 203.7 mm
- net /CLK': track 94.6 -> 84.7 mm
- net Net-(U3-K): track 16.9 -> 7.03 mm
- net Net-(U1A--): track 18.5 -> 8.97 mm
- net /B0': track 149.0 -> 156.6 mm
- net Net-(Q2A-E1): track 0.00 -> 6.48 mm
- net /B7': track 139.4 -> 133.2 mm
- net Net-(U2-R+): track 6.16 -> 0.00 mm
- net /B1': track 147.4 -> 153.2 mm
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Other:
- board text added: "*"
- board text added: "thismatters/turing-machine/v1"
- board text removed: "thismatters/turing-machine/v0"

Commit message: adding results from troubleshooting
Parts:
- added TP1: RAND, TestPoint:TestPoint_Plated_Hole_D2.0mm, B.Cu at (84.1, 51.8)
- added TP2: LOOP_CTRL, TestPoint:TestPoint_Plated_Hole_D2.0mm, B.Cu at (84.1, 56.4)
- C12: value 100n -> 1n
Routing:
- net /RAND': track 11.3 -> 27.1 mm
- net GND: track 341.7 -> 356.7 mm, vias 29 -> 30
- net /LOOP_CTRL': track 72.2 -> 76.8 mm
- net /_PULSE: track 51.8 -> 55.8 mm
- net /_CLK_LED: track 56.5 -> 57.0 mm

Commit message: v1a board ready, refit of v1 board available
Parts:
- removed R1, R2: 10, Resistor_SMD:R_0805_2012Metric
- added FB1: 70 Ohm, Inductor_SMD:L_0805_2012Metric, F.Cu at (61.2, 11.2)
- added FB2: 70 Ohm, Inductor_SMD:L_0805_2012Metric, F.Cu at (61.2, 8.89)
Other:
- board text added: "thismatters/turing-machine/v1a"
- board text removed: "thismatters/turing-machine/v1"
